File: SoundCard.kicad_pcb (KiCad board)
At the start: 2 copper layers, 79.5 x 51.7 mm, 18 parts, among them J1 AudioJack3, J2 Expansion / Diag Port, J3 Conn_Coaxial, U1 SN76489AN, U2 74LS11, U3 LM386, U4 74LS05, Y1 4Mhz

Commit message: Minor Changes
Parts:
- C1, C2: value C -> 10uf; footprint Capacitor_THT:C_Radial_D5.0mm_H5.0mm_P2.00mm -> Resistor_THT:R_Axial_DIN0204_L3.6mm_D1.6mm_P5.08mm_Horizontal
- R1: footprint Resistor_THT:R_Axial_DIN0414_L11.9mm_D4.5mm_P7.62mm_Vertical -> Resistor_THT:R_Axial_DIN0204_L3.6mm_D1.6mm_P5.08mm_Horizontal
- RV1: footprint Potentiometer_THT:Potentiometer_ACP_CA9-V10_Vertical_Hole -> Potentiometer_THT:Potentiometer_Bourns_3296W_Vertical
- moved RV1 7.74 mm to (198.0, 99.0)
Routing:
- net Net-(U1-AUDIO_OUT): track 58.6 -> 66.9 mm
- net Net-(U3-+): track 25.3 -> 19.2 mm

Commit message: x5
Routing:
- net D2: track 8.66 -> 9.56 mm
Other:
- board text added: "RETROLOGIC BY TOM SMITH v1 SOUND CARD"
Changed lines of the file:
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@@
 		(layer "Edge.Cuts")
+	)
+	(gr_text "RETROLOGIC\nBY TOM SMITH v1\nSOUND CARD"
+		(at 177.8508 66.8528 0)
+		(layer "F.SilkS")
+		(effects
+			(font
+				(size 1.5 1.5)
+				(thickness 0.3)
+				(bold yes)
+			)
+			(justify bottom)
+		)
 	)
 	(segment
@@
 	)
 	(segment
-		(start 130.6044 69.596)
+		(start 131.6918 68.5086)
+		(end 136.6872 68.5086)
+		(width 0.2)
+		(layer "B.Cu")
+		(net 19)
+	)
+	(segment
+		(start 129.5528 70.6476)
+		(end 131.6918 68.5086)
+		(width 0.2)
+		(layer "B.Cu")
+		(net 19)
+	)
+	(segment
+		(start 136.6872 68.5086)
 		(end 137.7746 69.596)
-		(width 0.2)
-		(layer "B.Cu")
-		(net 19)
-	)
-	(segment
-		(start 129.5528 70.6476)
-		(end 130.6044 69.596)
 		(width 0.2)
 		(layer "B.Cu")
@@
 	(segment
 		(start 155.7362 95.8254)
+		(end 149.5552 102.0064)
+		(width 0.2)
+		(layer "F.Cu")
+		(net 55)
+	)
+	(segment
+		(start 159.1056 91.2876)
+		(end 157.396 91.2876)
+		(width 0.2)
+		(layer "F.Cu")
+		(net 55)
+	)
+	(segment
+		(start 155.7362 92.9474)
+		(end 155.7362 95.8254)
+		(width 0.2)
+		(layer "F.Cu")
+		(net 55)
+	)
+	(segment
+		(start 157.396 91.2876)
 		(end 155.7362 92.9474)
 		(width 0.2)
@@
 		(net 55)
 	)
-	(segment
-		(start 155.7362 92.9474)
-		(end 154.5336 91.7448)
-		(width 0.2)
-		(layer "F.Cu")
-		(net 55)
-	)
-	(segment
-		(start 149.5552 102.0064)
-		(end 155.7362 95.8254)
-		(width 0.2)
-		(layer "F.Cu")
-		(net 55)
-	)
 	(via
-		(at 154.5336 91.7448)
+		(at 159.1056 91.2876)
 		(size 0.6)
 		(drill 0.3)
@@
 	)
 	(segment
+		(start 159.1056 87.1728)
+		(end 159.1514 87.127)
+		(width 0.2)
+		(layer "B.Cu")
+		(net 55)
+	)
+	(segment
+		(start 159.1056 91.2876)
+		(end 159.1056 87.1728)
+		(width 0.2)
+		(layer "B.Cu")
+		(net 55)
+	)
+	(segment
 		(start 159.1514 87.127)
 		(end 159.1514 86.5124)
 		(width 0.2)
 		(layer "B.Cu")
-		(net 55)
-	)
-	(segment
-		(start 154.5336 91.7448)
-		(end 159.1514 87.127)
-		(width 0.2)
-		(layer "B.Cu")
