File: 6502pc.kicad_pcb (KiCad board)
At the start: 2 copper layers, 145.6 x 96.2 mm, 45 parts, among them J1 DB9 Serial Port, J2 USB_B, J3 Port B, J4 Port A, J5 Display Connector, J6 SD-Card Board, J7 FTDI Socket, J9 Expansion / Diag Port, SW1 Reset Switch, SW2 SW_SPST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

Commit message: x
Parts:
- moved J9 3.91 mm to (155.9, 59.3)
Routing:
- net GND: track 66.5 -> 122.9 mm, vias 14 -> 10
- net A2: track 111.5 -> 164.4 mm, vias 0 -> 2
- net A1: track 139.7 -> 162.8 mm, vias 0 -> 1
- net D1: track 157.6 -> 137.4 mm, vias 3 -> 1
- net PA7: track 106.6 -> 125.9 mm, vias 1 -> 2
- net A7: track 92.4 -> 111.0 mm, vias 1 -> 5
- net Net-(U4-~{CS2}): track 108.7 -> 126.7 mm, vias 1 -> 2
- net PA4: track 185.3 -> 169.6 mm, vias 3 -> 2
- net PA0: track 55.2 -> 70.5 mm, vias 1 -> 0
- net D3: track 138.4 -> 153.5 mm
- net D2: track 153.0 -> 140.9 mm
- net Net-(D1-K): track 37.4 -> 49.0 mm
- net clock: track 248.3 -> 259.8 mm, vias 3 -> 2
- net Net-(J7-Pin_2): track 69.2 -> 58.4 mm, vias 2 -> 0
- net Net-(U3-~{CS}): track 35.4 -> 45.6 mm, vias 0 -> 1
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